Commit message: added k_ee_link

File: assets/urdf/franka_description/robots/franka_panda.urdf (robot description, URDF)
Before this commit: robot panda, 11 links, 10 joints
Links:
- added link k_ee_link
Joints:
- added joint k_ee: type fixed, parent panda_hand, child k_ee_link, origin xyz=0 0 0.103399 rpy=0 0 0
